Commit message: 修改了sensor_plugin中雷达支撑杆的长度

File: fishbot_description/urdf/fishbot/fishbot.urdf.xacro (robot description, xacro)
@@ -17,5 +17,5 @@
 <xacro:imu_xacro xyz="0.0 0.0 0.02"/>
 <xacro:camera_xacro xyz="0.10 0.0 0.075"/>
-<xacro:lidar_xacro xyz="0.0 0.0 0.10"/>
+<xacro:lidar_xacro xyz="0.0 0.0 0.15"/>
 <xacro:wheel_xacro wheel_name="left_wheel" xyz="0 0.10 -0.06"/>
 <xacro:wheel_xacro wheel_name="right_wheel" xyz="0 -0.10 -0.06"/>

File: fishbot_description/urdf/fishbot/sensor/lidar.urdf.xacro (robot description, xacro)
@@ -11,5 +11,5 @@
             <!-- 几何形状 -->
             <geometry>
-                <cylinder radius="0.01" length="0.10"/>
+                <cylinder radius="0.01" length="0.20"/>
             </geometry>
             <!-- 材质颜色 -->
@@ -63,5 +63,5 @@
      <!-- 机器人关节 -->
     <joint name="lidar_joint" type="fixed">
-        <origin xyz="0.0 0.0 0.05" rpy="0.0 0.0 0.0"/>
+        <origin xyz="0.0 0.0 0.1" rpy="0.0 0.0 0.0"/>
         <parent link="lidar_cylinder_link"/>
         <child link="lidar_link"/>

File: install/fishbot_description/share/fishbot_description/urdf/fishbot/plugins/gazebo_sensor_plugin.xacro (robot description, xacro)
@@ -20,5 +20,4 @@
                         <!-- 设置扫描范围 -->
                         <scan>
-                            <sphere radius="8.0"/>
                             <horizontal>
                                 <samples>360</samples>
